File: kicad/board-to-board.kicad_sch (KiCad schematic)
At the start: 6 parts, among them J8 DF40TC(3.0)-50DP-0.4V(51), J9 DF40TC(3.0)-50DP-0.4V(51)

Commit message: Update repo naming and cleanup files.
Signed-off-by: Benjamin Perseghetti <bperseghetti@rudislabs.com>
Other:
- title: MR-MCXN-T1 Sensor Node -> MR-MCXN-T1
Changed lines of the file:
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@@
 	(paper "A4")
 	(title_block
-		(title "MR-MCXN-T1 Sensor Node")
+		(title "MR-MCXN-T1")
 		(date "2025-03-28")
 		(rev "X0")
 		(company "NXP SEMICONDUCTORS B.V.")
-		(comment 1 "CLASSIFICATION: INTERNAL USE ONLY")
 		(comment 3 "DESIGNER: YOURI TILS")
 		(comment 4 "CTO SYSTEM INNOVATIONS / MOBILE ROBOTICS DOMAIN")
@@
 		)
 		(instances
-			(project "spinali_mcxn_t1_sensor_hub"
+			(project "spinali_mcxn_t1_hub"
 				(path "/8b469ec1-e800-4d46-8a32-95d77ceae6db/1eea4502-3ae6-49a1-b28d-d3586979946d"
 					(reference "#PWR0175")
@@
 		)
 		(instances
-			(project "spinali_mcxn_t1_sensor_hub"
+			(project "spinali_mcxn_t1_hub"
 				(path "/8b469ec1-e800-4d46-8a32-95d77ceae6db/1eea4502-3ae6-49a1-b28d-d3586979946d"
 					(reference "#PWR0196")
@@
 		)
 		(instances
-			(project "spinali_mcxn_t1_sensor_hub"
+			(project "spinali_mcxn_t1_hub"
 				(path "/8b469ec1-e800-4d46-8a32-95d77ceae6db/1eea4502-3ae6-49a1-b28d-d3586979946d"
 					(reference "#PWR0178")
@@
 		)
 		(instances
-			(project "spinali_mcxn_t1_sensor_hub"
+			(project "spinali_mcxn_t1_hub"
 				(path "/8b469ec1-e800-4d46-8a32-95d77ceae6db/1eea4502-3ae6-49a1-b28d-d3586979946d"
 					(reference "#PWR0237")
@@
 		)
 		(instances
-			(project "spinali_mcxn_t1_sensor_hub"
+			(project "spinali_mcxn_t1_hub"
 				(path "/8b469ec1-e800-4d46-8a32-95d77ceae6db/1eea4502-3ae6-49a1-b28d-d3586979946d"
 					(reference "#PWR0193")
@@
 		)
 		(instances
-			(project "spinali_mcxn_t1_sensor_hub"
+			(project "spinali_mcxn_t1_hub"
 				(path "/8b469ec1-e800-4d46-8a32-95d77ceae6db/1eea4502-3ae6-49a1-b28d-d3586979946d"
 					(reference "#PWR0190")
@@
 		)
 		(instances
-			(project "spinali_mcxn_t1_sensor_hub"
+			(project "spinali_mcxn_t1_hub"
 				(path "/8b469ec1-e800-4d46-8a32-95d77ceae6db/1eea4502-3ae6-49a1-b28d-d3586979946d"
 					(reference "#PWR0174")
@@
 		)
 		(instances
-			(project "spinali_mcxn_t1_sensor_hub"
+			(project "spinali_mcxn_t1_hub"
 				(path "/8b469ec1-e800-4d46-8a32-95d77ceae6db/1eea4502-3ae6-49a1-b28d-d3586979946d"
 					(reference "#PWR0198")
@@
 		)
 		(instances
-			(project "spinali_mcxn_t1_sensor_hub"
+			(project "spinali_mcxn_t1_hub"
 				(path "/8b469ec1-e800-4d46-8a32-95d77ceae6db/1eea4502-3ae6-49a1-b28d-d3586979946d"
 					(reference "#PWR0189")
@@
 		)
 		(instances
-			(project "spinali_mcxn_t1_sensor_hub"
+			(project "spinali_mcxn_t1_hub"
 				(path "/8b469ec1-e800-4d46-8a32-95d77ceae6db/1eea4502-3ae6-49a1-b28d-d3586979946d"
 					(reference "J8")
@@
 		)
 		(instances
-			(project "spinali_mcxn_t1_sensor_hub"
+			(project "spinali_mcxn_t1_hub"
 				(path "/8b469ec1-e800-4d46-8a32-95d77ceae6db/1eea4502-3ae6-49a1-b28d-d3586979946d"
 					(reference "#PWR0200")
@@
 		)
 		(instances
-			(project "spinali_mcxn_t1_sensor_hub"
+			(project "spinali_mcxn_t1_hub"
 				(path "/8b469ec1-e800-4d46-8a32-95d77ceae6db/1eea4502-3ae6-49a1-b28d-d3586979946d"
 					(reference "#PWR0185")
@@
 		)
 		(instances
-			(project "spinali_mcxn_t1_sensor_hub"
+			(project "spinali_mcxn_t1_hub"
 				(path "/8b469ec1-e800-4d46-8a32-95d77ceae6db/1eea4502-3ae6-49a1-b28d-d3586979946d"
 					(reference "#PWR0191")
@@
 		)
 		(instances
-			(project "spinali_mcxn_t1_sensor_hub"
+			(project "spinali_mcxn_t1_hub"
 				(path "/8b469ec1-e800-4d46-8a32-95d77ceae6db/1eea4502-3ae6-49a1-b28d-d3586979946d"
 					(reference "#PWR0179")
@@
 		)
 		(instances
-			(project "spinali_mcxn_t1_sensor_hub"
+			(project "spinali_mcxn_t1_hub"
 				(path "/8b469ec1-e800-4d46-8a32-95d77ceae6db/1eea4502-3ae6-49a1-b28d-d3586979946d"
 					(reference "#PWR0202")
@@
 		)
 		(instances
-			(project "spinali_mcxn_t1_sensor_hub"
+			(project "spinali_mcxn_t1_hub"
 				(path "/8b469ec1-e800-4d46-8a32-95d77ceae6db/1eea4502-3ae6-49a1-b28d-d3586979946d"
 					(reference "#PWR0197")
@@
 		)
 		(instances
-			(project "spinali_mcxn_t1_sensor_hub"
+			(project "spinali_mcxn_t1_hub"
 				(path "/8b469ec1-e800-4d46-8a32-95d77ceae6db/1eea4502-3ae6-49a1-b28d-d3586979946d"
 					(reference "#PWR0173")
@@
 		)
 		(instances
-			(project "spinali_mcxn_t1_sensor_hub"
+			(project "spinali_mcxn_t1_hub"
 				(path "/8b469ec1-e800-4d46-8a32-95d77ceae6db/1eea4502-3ae6-49a1-b28d-d3586979946d"
 					(reference "#PWR0181")
@@
 		)
 		(instances
-			(project "spinali_mcxn_t1_sensor_hub"
+			(project "spinali_mcxn_t1_hub"
 				(path "/8b469ec1-e800-4d46-8a32-95d77ceae6db/1eea4502-3ae6-49a1-b28d-d3586979946d"
 					(reference "#PWR0188")
@@
 		)
 		(instances
-			(project "spinali_mcxn_t1_sensor_hub"
+			(project "spinali_mcxn_t1_hub"
 				(path "/8b469ec1-e800-4d46-8a32-95d77ceae6db/1eea4502-3ae6-49a1-b28d-d3586979946d"
 					(reference "#PWR0192")
@@
 		)
 		(instances
-			(project "spinali_mcxn_t1_sensor_hub"
+			(project "spinali_mcxn_t1_hub"
 				(path "/8b469ec1-e800-4d46-8a32-95d77ceae6db/1eea4502-3ae6-49a1-b28d-d3586979946d"
 					(reference "#PWR0195")
@@
 		)
 		(instances
-			(project "spinali_mcxn_t1_sensor_hub"
+			(project "spinali_mcxn_t1_hub"
 				(path "/8b469ec1-e800-4d46-8a32-95d77ceae6db/1eea4502-3ae6-49a1-b28d-d3586979946d"
 					(reference "J9")
@@
 		)
 		(instances
-			(project "spinali_mcxn_t1_sensor_hub"
+			(project "spinali_mcxn_t1_hub"
 				(path "/8b469ec1-e800-4d46-8a32-95d77ceae6db/1eea4502-3ae6-49a1-b28d-d3586979946d"
 					(reference "#PWR0187")
@@
 		)
 		(instances
-			(project "spinali_mcxn_t1_sensor_hub"
+			(project "spinali_mcxn_t1_hub"
 				(path "/8b469ec1-e800-4d46-8a32-95d77ceae6db/1eea4502-3ae6-49a1-b28d-d3586979946d"
 					(reference "#PWR0235")
@@
 		)
 		(instances
-			(project "spinali_mcxn_t1_sensor_hub"
+			(project "spinali_mcxn_t1_hub"
 				(path "/8b469ec1-e800-4d46-8a32-95d77ceae6db/1eea4502-3ae6-49a1-b28d-d3586979946d"
 					(reference "#PWR0180")
@@
 		)
 		(instances
-			(project "spinali_mcxn_t1_sensor_hub"
+			(project "spinali_mcxn_t1_hub"
 				(path "/8b469ec1-e800-4d46-8a32-95d77ceae6db/1eea4502-3ae6-49a1-b28d-d3586979946d"
 					(reference "#PWR0199")
@@
 		)
 		(instances
-			(project "spinali_mcxn_t1_sensor_hub"
+			(project "spinali_mcxn_t1_hub"
 				(path "/8b469ec1-e800-4d46-8a32-95d77ceae6db/1eea4502-3ae6-49a1-b28d-d3586979946d"
 					(reference "#PWR0172")
@@
 		)
 		(instances
-			(project "spinali_mcxn_t1_sensor_hub"
+			(project "spinali_mcxn_t1_hub"
 				(path "/8b469ec1-e800-4d46-8a32-95d77ceae6db/1eea4502-3ae6-49a1-b28d-d3586979946d"
 					(reference "#PWR0236")
@@
 		)
 		(instances
-			(project "spinali_mcxn_t1_sensor_hub"
+			(project "spinali_mcxn_t1_hub"
 				(path "/8b469ec1-e800-4d46-8a32-95d77ceae6db/1eea4502-3ae6-49a1-b28d-d3586979946d"
 					(reference "#PWR0186")
@@
 		)
 		(instances
-			(project "spinali_mcxn_t1_sensor_hub"
+			(project "spinali_mcxn_t1_hub"
 				(path "/8b469ec1-e800-4d46-8a32-95d77ceae6db/1eea4502-3ae6-49a1-b28d-d3586979946d"
 					(reference "#PWR0184")
@@
 		)
 		(instances
-			(project "spinali_mcxn_t1_sensor_hub"
+			(project "spinali_mcxn_t1_hub"
 				(path "/8b469ec1-e800-4d46-8a32-95d77ceae6db/1eea4502-3ae6-49a1-b28d-d3586979946d"
 					(reference "#PWR0183")
@@
 		)
 		(instances
-			(project "spinali_mcxn_t1_sensor_hub"
+			(project "spinali_mcxn_t1_hub"
 				(path "/8b469ec1-e800-4d46-8a32-95d77ceae6db/1eea4502-3ae6-49a1-b28d-d3586979946d"
 					(reference "#PWR0238")
@@
 		)
 		(instances
-			(project "spinali_mcxn_t1_sensor_hub"
+			(project "spinali_mcxn_t1_hub"
 				(path "/8b469ec1-e800-4d46-8a32-95d77ceae6db/1eea4502-3ae6-49a1-b28d-d3586979946d"
 					(reference "#PWR0194")
@@
 		)
 		(instances
-			(project "spinali_mcxn_t1_sensor_hub"
+			(project "spinali_mcxn_t1_hub"
 				(path "/8b469ec1-e800-4d46-8a32-95d77ceae6db/1eea4502-3ae6-49a1-b28d-d3586979946d"
 					(reference "#PWR0177")
@@
 		)
 		(instances
-			(project "spinali_mcxn_t1_sensor_hub"
+			(project "spinali_mcxn_t1_hub"
 				(path "/8b469ec1-e800-4d46-8a32-95d77ceae6db/1eea4502-3ae6-49a1-b28d-d3586979946d"
 					(reference "#PWR0176")
@@
 		)
 		(instances
-			(project "spinali_mcxn_t1_sensor_hub"
+			(project "spinali_mcxn_t1_hub"
 				(path "/8b469ec1-e800-4d46-8a32-95d77ceae6db/1eea4502-3ae6-49a1-b28d-d3586979946d"
 					(reference "#PWR0201")
