File: kicad/communication.kicad_sch (KiCad schematic)
At the start: 34 parts, among them J10 SDO, J11 CKO, J12 GND, J3 CAN0A, J4 CAN0B, J5 Debug, J6 CAN1A, J7 CAN1B, U12 TJA1462ATK, U13 TJA1462ATK, U14 SK9822-EC20

Commit message: Updated layout and BOM
- Flipped Magnetometer so it is aligned with the axis of the IMU.
- Updated BOM so all parts can be sourced from DigiKey. Also added a row for JLCPCB part numbers if applicable.
- Replaced ISP button with the NanoT160AS. Added "ISP" in silkscreen at that button.
Parts:
- C67, C72: DigiKey (none) -> 490-6335-1-ND; JLCPCB (none) -> C77012; Supplier JLCPCB -> (none); Supplier PN C77012 -> (none)
- C68, C73, C77: DigiKey (none) -> 490-GRM155Z71A105KE01DCT-ND; JLCPCB (none) -> C528974; Supplier JLCPCB -> (none); Supplier PN C528974 -> (none)
- C69, C71, C74, C76: DigiKey (none) -> 311-1022-1-ND; JLCPCB (none) -> C107007; Supplier JLCPCB -> (none); Supplier PN C107007 -> (none)
- C70, C75: Supplier JLCPCB -> (none); Supplier PN C106208 -> (none)
- C78: DigiKey (none) -> 490-3261-1-ND; JLCPCB (none) -> C71629; MF Samsung Electro-Mechanics -> Murata Electronics; MFPN CL05B104KO5NNNC -> GRM155R71C104KA88D; Supplier JLCPCB -> (none); Supplier PN C1525 -> (none)
- D10, D11: DigiKey (none) -> 1727-7665-1-ND; JLCPCB (none) -> C552496; Supplier JLCPCB -> (none); Supplier PN C552496 -> (none)
- D8, D9: DigiKey (none) -> ESD7104MUTAGOSCT-ND; JLCPCB (none) -> C328026; Supplier JLCPCB -> (none); Supplier PN C328026 -> (none)
- J3, J4, J6, J7: DigiKey (none) -> 455-1566-1-ND; JLCPCB (none) -> C189895; Supplier JLCPCB -> (none); Supplier PN C189895 -> (none)
- J5: DigiKey (none) -> 455-SM10B-SRSS-TBCT-ND; JLCPCB (none) -> C160409; Supplier JLCPCB -> (none); Supplier PN C160409 -> (none)
- L6, L7: DigiKey (none) -> 541-IFLN1210BEER512NCT-ND; JLCPCB (none) -> -; Supplier DigiKey -> (none); Supplier PN 541-IFLN1210BEER512NCT-ND -> (none)
- R27, R28, R30, R31: Supplier DigiKey -> (none); Supplier PN 541-60.4SCT-ND -> (none)
- R29: DigiKey (none) -> YAG3561CT-ND; JLCPCB (none) -> C125923; MF UNI-ROYAL(Uniroyal Elec) -> YAGEO; MFPN 0603WAF1000T5E -> AC0603FR-07100RL; Supplier JLCPCB -> (none); Supplier PN C22775 -> (none)
- U12, U13: DigiKey (none) -> 568-TJA1462ATK/0ZCT-ND; Height 1 -> (none); JLCPCB (none) -> C3229259; MF NXP Semicon -> NXP USA Inc.; Manufacturer_Name NXP -> (none); Manufacturer_Part_Number TJA1462ATK -> (none); Supplier JLCPCB -> (none); Supplier PN C3229259 -> (none)
- U14: DigiKey (none) -> 2007-BB-2020BGR-TRBCT-ND; Height 0.75 -> (none); JLCPCB (none) -> C2909059; Manufacturer_Name DONGGUAN OPSCO OPTOELECTRONICS CO., LTD -> (none); Manufacturer_Part_Number SK9822-EC20 -> (none); Supplier JLCPCB -> (none); Supplier PN C2909059 -> (none)

Commit message: Update repo naming and cleanup files.
Signed-off-by: Benjamin Perseghetti <bperseghetti@rudislabs.com>
Other:
- title: MR-MCXN-T1 Sensor Node -> MR-MCXN-T1

Commit message: Patched schematic and board layout
- Replaced choke in series with Vbus with 2A choke.
- Fixed interface to the BMP581 barometer.
- Added schematic fixes to the layout.
- Completed DRC.
- Created production folder with Gerber, BOM, positions and schematic.
Parts:
- C70, C75: DigiKey (none) -> 311-1418-1-ND
- R27, R28, R30, R31: DigiKey (none) -> 541-60.4SCT-ND
Changed lines of the file:
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@@
 (kicad_sch
-	(version 20231120)
+	(version 20250114)
 	(generator "eeschema")
-	(generator_version "8.0")
+	(generator_version "9.0")
 	(paper "A4")
 	(title_block
@@
 		(comment 4 "CTO SYSTEM INNOVATIONS / MOBILE ROBOTICS DOMAIN")
 	)
+	(text "Drive CANx_STB LOW\nto enable CAN transceiver"
+		(exclude_from_sim no)
+		(at 136.906 76.2 0)
+		(effects
+			(font
+				(size 1.27 1.27)
+			)
+		)
+	)
+	(text "Drive CANx_STB LOW\nto enable CAN transceiver"
+		(exclude_from_sim no)
+		(at 135.89 136.144 0)
+		(effects
+			(font
+				(size 1.27 1.27)
+			)
+		)
+	)
 	(junction
 		(at 238.76 135.89)
@@
 		)
 	)
-	(text "Drive CANx_STB LOW\nto enable CAN transceiver"
-		(exclude_from_sim no)
-		(at 136.906 76.2 0)
-		(effects
-			(font
-				(size 1.27 1.27)
-			)
-		)
-	)
-	(text "Drive CANx_STB LOW\nto enable CAN transceiver"
-		(exclude_from_sim no)
-		(at 135.89 136.144 0)
-		(effects
-			(font
-				(size 1.27 1.27)
-			)
-		)
-	)
 	(global_label "P4_14{slash}CAN0_STB"
 		(shape bidirectional)
@@
 			)
 		)
+		(property "DigiKey" "541-60.4SCT-ND"
+			(at 212.09 120.65 0)
+			(effects
+				(font
+					(size 1.27 1.27)
+				)
+				(hide yes)
+			)
+		)
 		(pin "1"
 		)
@@
 			)
 		)
+		(property "DigiKey" "541-60.4SCT-ND"
+			(at 212.09 71.12 0)
+			(effects
+				(font
+					(size 1.27 1.27)
+				)
+				(hide yes)
+			)
+		)
 		(pin "1"
 		)
@@
 			)
 		)
+		(property "DigiKey" "541-60.4SCT-ND"
+			(at 212.09 130.81 0)
+			(effects
+				(font
+					(size 1.27 1.27)
+				)
+				(hide yes)
+			)
+		)
 		(pin "1"
 		)
@@
 			)
 		)
+		(property "DigiKey" "541-60.4SCT-ND"
+			(at 212.09 60.96 0)
+			(effects
+				(font
+					(size 1.27 1.27)
+				)
+				(hide yes)
+			)
+		)
 		(pin "1"
 		)
@@
 			)
 		)
+		(property "DigiKey" "311-1418-1-ND"
+			(at 207.01 66.04 90)
+			(effects
+				(font
+					(size 1.27 1.27)
+				)
+				(hide yes)
+			)
+		)
 		(pin "2"
 		)
@@
 			(effects
 				(font
+					(size 1.27 1.27)
+				)
+				(hide yes)
+			)
+		)
+		(property "DigiKey" "311-1418-1-ND"
+			(at 207.01 125.73 90)
+			(effects
+				(font
