File: kicad/mcu_io_1.kicad_sch (KiCad schematic)
At the start: 11 parts, among them SW1 ISP, U7 MCXN947VDFT, Y1 24MHz

Commit message: Update repo naming and cleanup files.
Signed-off-by: Benjamin Perseghetti <bperseghetti@rudislabs.com>
Other:
- title: MR-MCXN-T1 Sensor Node -> MR-MCXN-T1
Changed lines of the file:
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@@
 	(paper "A3")
 	(title_block
-		(title "MR-MCXN-T1 Sensor Node")
+		(title "MR-MCXN-T1")
 		(date "2025-03-28")
 		(rev "X0")
 		(company "NXP SEMICONDUCTORS B.V.")
-		(comment 1 "CLASSIFICATION: INTERNAL USE ONLY")
 		(comment 3 "DESIGNER: YOURI TILS")
 		(comment 4 "CTO SYSTEM INNOVATIONS / MOBILE ROBOTICS DOMAIN")
@@
 		)
 		(instances
-			(project "spinali_mcxn_t1_sensor_hub"
+			(project "spinali_mcxn_t1_hub"
 				(path "/8b469ec1-e800-4d46-8a32-95d77ceae6db/2f800241-08a7-49e7-97bc-35e3807b9c21"
 					(reference "#PWR053")
@@
 		)
 		(instances
-			(project "spinali_mcxn_t1_sensor_hub"
+			(project "spinali_mcxn_t1_hub"
 				(path "/8b469ec1-e800-4d46-8a32-95d77ceae6db/2f800241-08a7-49e7-97bc-35e3807b9c21"
 					(reference "#PWR048")
@@
 		)
 		(instances
-			(project "spinali_mcxn_t1_sensor_hub"
+			(project "spinali_mcxn_t1_hub"
 				(path "/8b469ec1-e800-4d46-8a32-95d77ceae6db/2f800241-08a7-49e7-97bc-35e3807b9c21"
 					(reference "#PWR052")
@@
 		)
 		(instances
-			(project "spinali_mcxn_t1_sensor_hub"
+			(project "spinali_mcxn_t1_hub"
 				(path "/8b469ec1-e800-4d46-8a32-95d77ceae6db/2f800241-08a7-49e7-97bc-35e3807b9c21"
 					(reference "#PWR051")
@@
 		)
 		(instances
-			(project "spinali_mcxn_t1_sensor_hub"
+			(project "spinali_mcxn_t1_hub"
 				(path "/8b469ec1-e800-4d46-8a32-95d77ceae6db/2f800241-08a7-49e7-97bc-35e3807b9c21"
 					(reference "#PWR054")
@@
 		)
 		(instances
-			(project "spinali_mcxn_t1_sensor_hub"
+			(project "spinali_mcxn_t1_hub"
 				(path "/8b469ec1-e800-4d46-8a32-95d77ceae6db/2f800241-08a7-49e7-97bc-35e3807b9c21"
 					(reference "#PWR050")
@@
 		)
 		(instances
-			(project "spinali_mcxn_t1_sensor_hub"
+			(project "spinali_mcxn_t1_hub"
 				(path "/8b469ec1-e800-4d46-8a32-95d77ceae6db/2f800241-08a7-49e7-97bc-35e3807b9c21"
 					(reference "R18")
@@
 		)
 		(instances
-			(project "spinali_mcxn_t1_sensor_hub"
+			(project "spinali_mcxn_t1_hub"
 				(path "/8b469ec1-e800-4d46-8a32-95d77ceae6db/2f800241-08a7-49e7-97bc-35e3807b9c21"
 					(reference "R19")
@@
 		)
 		(instances
-			(project "spinali_mcxn_t1_sensor_hub"
+			(project "spinali_mcxn_t1_hub"
 				(path "/8b469ec1-e800-4d46-8a32-95d77ceae6db/2f800241-08a7-49e7-97bc-35e3807b9c21"
 					(reference "#PWR055")

Commit message: Patched schematic and board layout
- Replaced choke in series with Vbus with 2A choke.
- Fixed interface to the BMP581 barometer.
- Added schematic fixes to the layout.
- Completed DRC.
- Created production folder with Gerber, BOM, positions and schematic.
Parts:
- R16, R17, R18, R19: DigiKey (none) -> YAG3436CT-ND; JLCPCB (none) -> C144807; MF UNI-ROYAL(Uniroyal Elec) -> YAGEO; MFPN 0402WGF1002TCE -> AC0402FR-0710KL
- R20: DigiKey (none) -> YAG3450CT-ND; MF UNI-ROYAL(Uniroyal Elec) -> YAGEO; MFPN 0402WGF1004TCE -> AC0402FR-071ML
Changed lines of the file:
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@@
 (kicad_sch
-	(version 20231120)
+	(version 20250114)
 	(generator "eeschema")
-	(generator_version "8.0")
+	(generator_version "9.0")
 	(paper "A3")
 	(title_block
@@
 			)
 		)
-		(property "MF" "UNI-ROYAL(Uniroyal Elec)"
+		(property "MF" "YAGEO"
+			(at 57.15 138.43 0)
+			(effects
+				(font
+					(size 1.27 1.27)
+				)
+				(hide yes)
+			)
+		)
+		(property "MFPN" "AC0402FR-0710KL"
+			(at 57.15 138.43 0)
+			(effects
+				(font
+					(size 1.27 1.27)
+				)
+				(hide yes)
+			)
+		)
+		(property "DigiKey" "YAG3436CT-ND"
 			(at 57.15 138.43 0)
 			(effects
@@
 			)
 		)
-		(property "MFPN" "0402WGF1002TCE"
+		(property "JLCPCB" "C144807"
 			(at 57.15 138.43 0)
 			(effects
@@
 			)
 		)
-		(property "MF" "UNI-ROYAL(Uniroyal Elec)"
+		(property "MF" "YAGEO"
+			(at 48.26 68.58 0)
+			(effects
+				(font
+					(size 1.27 1.27)
+				)
+				(hide yes)
+			)
+		)
+		(property "MFPN" "AC0402FR-0710KL"
+			(at 48.26 68.58 0)
+			(effects
+				(font
+					(size 1.27 1.27)
+				)
+				(hide yes)
+			)
+		)
+		(property "DigiKey" "YAG3436CT-ND"
 			(at 48.26 68.58 0)
 			(effects
@@
 			)
 		)
-		(property "MFPN" "0402WGF1002TCE"
+		(property "JLCPCB" "C144807"
 			(at 48.26 68.58 0)
 			(effects
@@
 			)
 		)
-		(property "MF" "UNI-ROYAL(Uniroyal Elec)"
+		(property "MF" "YAGEO"
+			(at 57.15 68.58 0)
+			(effects
+				(font
+					(size 1.27 1.27)
+				)
+				(hide yes)
+			)
+		)
+		(property "MFPN" "AC0402FR-0710KL"
+			(at 57.15 68.58 0)
+			(effects
+				(font
+					(size 1.27 1.27)
+				)
+				(hide yes)
+			)
+		)
+		(property "DigiKey" "YAG3436CT-ND"
 			(at 57.15 68.58 0)
 			(effects
@@
 			)
 		)
-		(property "MFPN" "0402WGF1002TCE"
+		(property "JLCPCB" "C144807"
 			(at 57.15 68.58 0)
 			(effects
@@
 			)
 		)
-		(property "MF" "UNI-ROYAL(Uniroyal Elec)"
+		(property "MF" "YAGEO"
 			(at 49.53 194.31 0)
 			(effects
@@
 			)
 		)
-		(property "MFPN" "0402WGF1004TCE"
+		(property "MFPN" "AC0402FR-071ML"
 			(at 49.53 194.31 0)
 			(effects
@@
 			)
 		)
+		(property "DigiKey" "YAG3450CT-ND"
+			(at 49.53 194.31 90)
+			(effects
+				(font
+					(size 1.27 1.27)
+				)
+				(hide yes)
+			)
+		)
 		(pin "2"
 		)
@@
 			)
 		)
-		(property "MF" "UNI-ROYAL(Uniroyal Elec)"
+		(property "MF" "YAGEO"
+			(at 66.04 138.43 0)
+			(effects
+				(font
+					(size 1.27 1.27)
+				)
+				(hide yes)
+			)
+		)
+		(property "MFPN" "AC0402FR-0710KL"
 			(at 66.04 138.43 0)
 			(effects
@@
 			)
 		)
-		(property "MFPN" "0402WGF1002TCE"
+		(property "DigiKey" "YAG3436CT-ND"
+			(at 66.04 138.43 0)
+			(effects
+				(font
+					(size 1.27 1.27)
+				)
+				(hide yes)
+			)
+		)
+		(property "JLCPCB" "C144807"
 			(at 66.04 138.43 0)
 			(effects
