File: kicad/ethernet_phy.kicad_sch (KiCad schematic)
At the start: 41 parts, among them U15 TJA1103AHN, Y3 25MHz

Commit message: MR-MCXN-T1 Rev A Production
- Added Rev A in schematic and layout
- Updated footprints
- Succesfull DRC

Signed-off-by: Youri Tils <youri.tils@nxp.com>
Other:
- company: NXP SEMICONDUCTORS B.V. -> ${COMPANY}
- title: MR-MCXN-T1 -> ${TITLE}
Changed lines of the file:
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@@
 	(paper "A3")
 	(title_block
-		(title "MR-MCXN-T1")
-		(date "2026-07-27")
-		(rev "X1")
-		(company "NXP SEMICONDUCTORS B.V.")
-		(comment 1 "DESIGNER: YOURI TILS")
-		(comment 2 "CTO SYSTEM INNOVATIONS / MOBILE ROBOTICS DOMAIN")
+		(title "${TITLE}")
+		(date "2026-08-24")
+		(rev "${BOARD_REV}")
+		(company "${COMPANY}")
+		(comment 1 "DESIGNER: ${DESIGNER}")
+		(comment 2 "${DEPARTMENT}")
+		(comment 3 "REVIEWED BY: ${REVIEWER}")
 	)
 	(text "CONFIG0 = LOW, CONFIG1 = OPEN, CONFIG2 = OPEN \nSelects PHYAD = 18"
@@
 		)
 		(instances
-			(project ""
+			(project "spinali_mcxn_t1_hub"
 				(path "/8b469ec1-e800-4d46-8a32-95d77ceae6db/a20b3bd6-c7b2-46ff-9591-ca80b372e5a4"
 					(reference "D14")
@@
 		)
 		(instances
-			(project ""
+			(project "spinali_mcxn_t1_hub"
 				(path "/8b469ec1-e800-4d46-8a32-95d77ceae6db/a20b3bd6-c7b2-46ff-9591-ca80b372e5a4"
 					(reference "R46")
@@
 		)
 		(instances
-			(project ""
+			(project "spinali_mcxn_t1_hub"
 				(path "/8b469ec1-e800-4d46-8a32-95d77ceae6db/a20b3bd6-c7b2-46ff-9591-ca80b372e5a4"
 					(reference "R34")
@@
 		)
 		(instances
-			(project ""
+			(project "spinali_mcxn_t1_hub"
 				(path "/8b469ec1-e800-4d46-8a32-95d77ceae6db/a20b3bd6-c7b2-46ff-9591-ca80b372e5a4"
 					(reference "R43")
@@
 		)
 		(instances
-			(project ""
+			(project "spinali_mcxn_t1_hub"
 				(path "/8b469ec1-e800-4d46-8a32-95d77ceae6db/a20b3bd6-c7b2-46ff-9591-ca80b372e5a4"
 					(reference "L10")
@@
 		)
 		(instances
-			(project ""
+			(project "spinali_mcxn_t1_hub"
 				(path "/8b469ec1-e800-4d46-8a32-95d77ceae6db/a20b3bd6-c7b2-46ff-9591-ca80b372e5a4"
 					(reference "R33")
