File: kicad/mcu_io_2.kicad_sch (KiCad schematic)
At the start: 4 parts, among them U7 MCXN947VDFT, Y2 32.768kHz

Commit message: MR-MCXN-T1 Rev A Production
- Added Rev A in schematic and layout
- Updated footprints
- Succesfull DRC

Signed-off-by: Youri Tils <youri.tils@nxp.com>
Other:
- company: NXP SEMICONDUCTORS B.V. -> ${COMPANY}
- title: MR-MCXN-T1 -> ${TITLE}
Changed lines of the file:
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@@
 	(paper "A3")
 	(title_block
-		(title "MR-MCXN-T1")
-		(date "2026-07-27")
-		(rev "X1")
-		(company "NXP SEMICONDUCTORS B.V.")
-		(comment 1 "DESIGNER: YOURI TILS")
-		(comment 2 "CTO SYSTEM INNOVATIONS / MOBILE ROBOTICS DOMAIN")
+		(title "${TITLE}")
+		(date "2026-08-24")
+		(rev "${BOARD_REV}")
+		(company "${COMPANY}")
+		(comment 1 "DESIGNER: ${DESIGNER}")
+		(comment 2 "${DEPARTMENT}")
+		(comment 3 "REVIEWED BY: ${REVIEWER}")
 	)
 	(junction
@@
 		)
 		(instances
-			(project ""
+			(project "spinali_mcxn_t1_hub"
 				(path "/8b469ec1-e800-4d46-8a32-95d77ceae6db/4619e5be-1f0d-457d-96e5-6e6d95033c83"
 					(reference "C27")
@@
 		)
 		(instances
-			(project ""
+			(project "spinali_mcxn_t1_hub"
 				(path "/8b469ec1-e800-4d46-8a32-95d77ceae6db/4619e5be-1f0d-457d-96e5-6e6d95033c83"
 					(reference "Y2")
@@
 		)
 		(instances
-			(project ""
+			(project "spinali_mcxn_t1_hub"
 				(path "/8b469ec1-e800-4d46-8a32-95d77ceae6db/4619e5be-1f0d-457d-96e5-6e6d95033c83"
 					(reference "#PWR057")
@@
 		)
 		(instances
-			(project ""
+			(project "spinali_mcxn_t1_hub"
 				(path "/8b469ec1-e800-4d46-8a32-95d77ceae6db/4619e5be-1f0d-457d-96e5-6e6d95033c83"
 					(reference "U7")
@@
 		)
 		(instances
-			(project ""
+			(project "spinali_mcxn_t1_hub"
 				(path "/8b469ec1-e800-4d46-8a32-95d77ceae6db/4619e5be-1f0d-457d-96e5-6e6d95033c83"
 					(reference "U7")
@@
 		)
 		(instances
-			(project ""
+			(project "spinali_mcxn_t1_hub"
 				(path "/8b469ec1-e800-4d46-8a32-95d77ceae6db/4619e5be-1f0d-457d-96e5-6e6d95033c83"
 					(reference "C28")
@@
 		)
 		(instances
-			(project ""
+			(project "spinali_mcxn_t1_hub"
 				(path "/8b469ec1-e800-4d46-8a32-95d77ceae6db/4619e5be-1f0d-457d-96e5-6e6d95033c83"
 					(reference "#PWR056")
@@
 		)
 		(instances
-			(project ""
+			(project "spinali_mcxn_t1_hub"
 				(path "/8b469ec1-e800-4d46-8a32-95d77ceae6db/4619e5be-1f0d-457d-96e5-6e6d95033c83"
 					(reference "U7")
