File: kicad/mcu_usb_power.kicad_sch (KiCad schematic)
At the start: 44 parts, among them J2 USB4105-GF-A, U7 MCXN947VDFT, U8 PCMF1USB3SZ

Commit message: MR-MCXN-T1 Rev A Production
- Added Rev A in schematic and layout
- Updated footprints
- Succesfull DRC

Signed-off-by: Youri Tils <youri.tils@nxp.com>
Other:
- company: NXP SEMICONDUCTORS B.V. -> ${COMPANY}
- title: MR-MCXN-T1 -> ${TITLE}
Changed lines of the file:
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@@
 	(paper "A3")
 	(title_block
-		(title "MR-MCXN-T1")
-		(date "2026-07-27")
-		(rev "X1")
-		(company "NXP SEMICONDUCTORS B.V.")
-		(comment 1 "DESIGNER: YOURI TILS")
-		(comment 2 "CTO SYSTEM INNOVATIONS / MOBILE ROBOTICS DOMAIN")
+		(title "${TITLE}")
+		(date "2026-08-24")
+		(rev "${BOARD_REV}")
+		(company "${COMPANY}")
+		(comment 1 "DESIGNER: ${DESIGNER}")
+		(comment 2 "${DEPARTMENT}")
+		(comment 3 "REVIEWED BY: ${REVIEWER}")
 	)
 	(text "Place close to VDD"
@@
 		)
 		(instances
-			(project ""
+			(project "spinali_mcxn_t1_hub"
 				(path "/8b469ec1-e800-4d46-8a32-95d77ceae6db/cb14c3cb-ad07-49c0-85e6-22786ebb10ed"
 					(reference "#PWR094")
@@
 		)
 		(instances
-			(project ""
+			(project "spinali_mcxn_t1_hub"
 				(path "/8b469ec1-e800-4d46-8a32-95d77ceae6db/cb14c3cb-ad07-49c0-85e6-22786ebb10ed"
 					(reference "R21")
@@
 		)
 		(instances
-			(project ""
+			(project "spinali_mcxn_t1_hub"
 				(path "/8b469ec1-e800-4d46-8a32-95d77ceae6db/cb14c3cb-ad07-49c0-85e6-22786ebb10ed"
 					(reference "U7")
@@
 		)
 		(instances
-			(project "flow_max"
+			(project "spinali_mcxn_t1_hub"
 				(path "/8b469ec1-e800-4d46-8a32-95d77ceae6db/cb14c3cb-ad07-49c0-85e6-22786ebb10ed"
 					(reference "#PWR0104")
@@
 		)
 		(instances
-			(project "flow_max"
+			(project "spinali_mcxn_t1_hub"
 				(path "/8b469ec1-e800-4d46-8a32-95d77ceae6db/cb14c3cb-ad07-49c0-85e6-22786ebb10ed"
 					(reference "#PWR097")
@@
 		)
 		(instances
-			(project ""
+			(project "spinali_mcxn_t1_hub"
 				(path "/8b469ec1-e800-4d46-8a32-95d77ceae6db/cb14c3cb-ad07-49c0-85e6-22786ebb10ed"
 					(reference "U7")
@@
 		)
 		(instances
-			(project ""
+			(project "spinali_mcxn_t1_hub"
 				(path "/8b469ec1-e800-4d46-8a32-95d77ceae6db/cb14c3cb-ad07-49c0-85e6-22786ebb10ed"
 					(reference "U8")
@@
 		)
 		(instances
-			(project ""
+			(project "spinali_mcxn_t1_hub"
 				(path "/8b469ec1-e800-4d46-8a32-95d77ceae6db/cb14c3cb-ad07-49c0-85e6-22786ebb10ed"
 					(reference "J2")
@@
 		)
 		(instances
-			(project ""
+			(project "spinali_mcxn_t1_hub"
 				(path "/8b469ec1-e800-4d46-8a32-95d77ceae6db/cb14c3cb-ad07-49c0-85e6-22786ebb10ed"
 					(reference "C48")
@@
 		)
 		(instances
-			(project ""
+			(project "spinali_mcxn_t1_hub"
 				(path "/8b469ec1-e800-4d46-8a32-95d77ceae6db/cb14c3cb-ad07-49c0-85e6-22786ebb10ed"
 					(reference "C56")
@@
 		)
 		(instances
-			(project ""
+			(project "spinali_mcxn_t1_hub"
 				(path "/8b469ec1-e800-4d46-8a32-95d77ceae6db/cb14c3cb-ad07-49c0-85e6-22786ebb10ed"
 					(reference "#PWR0101")
@@
 		)
 		(instances
-			(project ""
+			(project "spinali_mcxn_t1_hub"
 				(path "/8b469ec1-e800-4d46-8a32-95d77ceae6db/cb14c3cb-ad07-49c0-85e6-22786ebb10ed"
 					(reference "L3")
@@
 		)
 		(instances
-			(project ""
+			(project "spinali_mcxn_t1_hub"
 				(path "/8b469ec1-e800-4d46-8a32-95d77ceae6db/cb14c3cb-ad07-49c0-85e6-22786ebb10ed"
 					(reference "C59")
@@
 		)
 		(instances
-			(project ""
+			(project "spinali_mcxn_t1_hub"
 				(path "/8b469ec1-e800-4d46-8a32-95d77ceae6db/cb14c3cb-ad07-49c0-85e6-22786ebb10ed"
 					(reference "D7")
@@
 		)
 		(instances
-			(project ""
+			(project "spinali_mcxn_t1_hub"
 				(path "/8b469ec1-e800-4d46-8a32-95d77ceae6db/cb14c3cb-ad07-49c0-85e6-22786ebb10ed"
 					(reference "R25")
@@
 		)
 		(instances
-			(project ""
+			(project "spinali_mcxn_t1_hub"
 				(path "/8b469ec1-e800-4d46-8a32-95d77ceae6db/cb14c3cb-ad07-49c0-85e6-22786ebb10ed"
 					(reference "L4")
@@
 		)
 		(instances
-			(project "flow_max"
+			(project "spinali_mcxn_t1_hub"
 				(path "/8b469ec1-e800-4d46-8a32-95d77ceae6db/cb14c3cb-ad07-49c0-85e6-22786ebb10ed"
 					(reference "#PWR095")
@@
 		)
 		(instances
-			(project ""
+			(project "spinali_mcxn_t1_hub"
 				(path "/8b469ec1-e800-4d46-8a32-95d77ceae6db/cb14c3cb-ad07-49c0-85e6-22786ebb10ed"
 					(reference "D6")
@@
 		)
 		(instances
-			(project "flow_max"
+			(project "spinali_mcxn_t1_hub"
 				(path "/8b469ec1-e800-4d46-8a32-95d77ceae6db/cb14c3cb-ad07-49c0-85e6-22786ebb10ed"
 					(reference "#PWR080")
