File: kicad/block_diagram_sch.kicad_sch (KiCad schematic)
At the start: 0 parts

Commit message: Updated Block diagram
Signed-off-by: Youri Tils <youri.tils@nxp.com>
Other:
- note added: "3.3V"
- note added: "5V"
- note added: "Board-To-Board Connector 1"
- note added: "Board-To-Board Connector 2"
- note added: "CAN Connector"
- note added: "CAN FD PHY"
- note added: "DF40TC"
- note added: "FLEXCOMM1_UART / DEBUG_SWD"
- note added: "FLEXCOMM8_SPI"
- note added: "FLEXIO"
- note added: "GPIO 4x FLEXCOMM FLEXIO SmartDMA SDHC0 ADC COMPARATOR FLEXPWM SAI PDM"
- note added: "I3C0"
- note added: "Input connector Power 3S-12S + 100Base-T1"
- note added: "Load switch NX5P3363UKZ"
- note added: "Micro Lock Plus"
- note added: "Pixhawk Debug Full Connector"
- note added: "RMII"
- note added: "Reverse polarity protection + DCDC"
- note added: "VBAT"
- note added: "VBAT RTC 5.0V 1A 3.3V 500mA 1.8V 200mA I3C1 GPIO 3x FLEXCOMM FLEXIO SmartDMA ADC COMPARATOR OPAMP DAC FLEXPWM"
- note removed: "+60V Max"
- note removed: "5V 3V"
- note removed: "Ancillary to core functionality"
- note removed: "CAN-FD"
- note removed: "ETH"
- note removed: "GPIO SDHC0 SmartDMA FLEXCOMM0 FLEXCOMM3 FLEXCOMM7 FLEXIO"
- note removed: "I3C"
- note removed: "J8"
- note removed: "J9"
- note removed: "SPI"
- note removed: "Unified 100BaseT1 and VBatt <60V connnector"
- note removed: "Vbatt 5.0V 3.3V 1.8V I3C (I2C) GPIO FLEXCOMM2 FLEXCOMM4 FLEXCOMM6 FLEXIO_0 Analog OPAMP DAC"
